File: Gregory.kicad_sch (KiCad schematic)
At the start: 37 parts, among them J1 Conn_01x03_Pin, SW1 SW_Push, SW10 SW_Push, SW11 SW_Push, SW12 SW_Push, SW13 SW_Push, SW14 SW_Push, SW15 SW_Push, SW16 SW_Push, SW17 RotaryEncoder, SW2 SW_Push, SW3 SW_Push, SW4 SW_Push, SW5 SW_Push, SW6 SW_Push, SW7 SW_Push, SW8 SW_Push, SW9 SW_Push, U1 MOUDLE-SEEEDUINO-XIAO, U2 ER_OLEDM0.91_1x-I2C

Commit message: Add files via upload
Parts:
- added TP1, TP2, TP3, TP4, TP5, TP6: TestPoint, TestPoint:TestPoint_Pad_D1.5mm, symbol Connector:TestPoint
Connections:
- net 5V: now also TP2.1, TP5.1
- net GND: now also TP1.1, TP6.1
- net I2C_SCL: now also U1.6 (PA9_A5_D5_SCL), TP4.1; no longer U1.5 (PA8_A4_D4_SDA)
- net I2C_SDA: now also U1.5 (PA8_A4_D4_SDA), TP3.1; no longer U1.6 (PA9_A5_D5_SCL)

Commit message: Add files via upload
Connections:
- net Row2: no longer D17.1 (K)
- net Row3: now also D17.1 (K)
Changed lines of the file:
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@@
 		)
 	)
-	(label "Row2"
+	(label "Row3"
 		(at 214.63 35.56 0)
 		(effects

Commit message: Add files via upload
Parts:
- added D18: 1N4148, Diode_THT:D_DO-35_SOD27_P7.62mm_Horizontal, symbol Diode:1N4148
Connections:
- net Column0: now also D17.1 (K); no longer SW17.A
- net Column1: now also D18.1 (K); no longer SW17.B
- net Row0: now also SW17.C
- net Row3: no longer D17.1 (K)
- net at D17.2 (A): now also SW17.A; no longer SW17.C
- new net: D18.2 (A), SW17.B
Other:
- moved on the sheet: D17
Changed lines of the file:
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@@
 	(wire
 		(pts
+			(xy 222.25 38.1) (xy 222.25 41.91)
+		)
+		(stroke
+			(width 0)
+			(type default)
+		)
+	)
+	(wire
+		(pts
 			(xy 119.38 81.28) (xy 119.38 99.06)
 		)
@@
 	(wire
 		(pts
-			(xy 224.79 33.02) (xy 231.14 33.02)
+			(xy 31.75 95.25) (xy 34.29 95.25)
 		)
 		(stroke
@@
 	(wire
 		(pts
-			(xy 31.75 95.25) (xy 34.29 95.25)
+			(xy 31.75 100.33) (xy 34.29 100.33)
 		)
 		(stroke
@@
 	(wire
 		(pts
-			(xy 31.75 100.33) (xy 34.29 100.33)
+			(xy 119.38 63.5) (xy 151.13 63.5)
 		)
 		(stroke
@@
 	(wire
 		(pts
-			(xy 119.38 63.5) (xy 151.13 63.5)
+			(xy 146.05 60.96) (xy 166.37 60.96)
 		)
 		(stroke
@@
 	(wire
 		(pts
-			(xy 146.05 60.96) (xy 166.37 60.96)
+			(xy 166.37 60.96) (xy 186.69 60.96)
 		)
 		(stroke
@@
 	(wire
 		(pts
-			(xy 166.37 60.96) (xy 186.69 60.96)
+			(xy 119.38 46.99) (xy 151.13 46.99)
 		)
 		(stroke
@@
 	(wire
 		(pts
-			(xy 119.38 46.99) (xy 151.13 46.99)
+			(xy 101.6 88.9) (xy 102.87 88.9)
 		)
 		(stroke
@@
 	(wire
 		(pts
-			(xy 101.6 88.9) (xy 102.87 88.9)
+			(xy 229.87 38.1) (xy 231.14 38.1)
 		)
 		(stroke
@@
 	(wire
 		(pts
-			(xy 226.06 35.56) (xy 231.14 35.56)
-		)
-		(stroke
-			(width 0)
-			(type default)
-		)
-	)
-	(wire
-		(pts
 			(xy 166.37 96.52) (xy 186.69 96.52)
 		)
@@
 	(wire
 		(pts
-			(xy 224.79 38.1) (xy 231.14 38.1)
+			(xy 171.45 44.45) (xy 224.79 44.45)
 		)
 		(stroke
@@
 	(wire
 		(pts
-			(xy 171.45 44.45) (xy 224.79 44.45)
+			(xy 191.77 66.04) (xy 214.63 66.04)
 		)
 		(stroke
@@
 	(wire
 		(pts
-			(xy 191.77 66.04) (xy 214.63 66.04)
+			(xy 172.72 33.02) (xy 179.07 33.02)
 		)
 		(stroke
@@
 	(wire
 		(pts
-			(xy 172.72 33.02) (xy 179.07 33.02)
+			(xy 224.79 35.56) (xy 231.14 35.56)
 		)
 		(stroke
@@
 	(wire
 		(pts
+			(xy 222.25 29.21) (xy 222.25 33.02)
+		)
+		(stroke
+			(width 0)
+			(type default)
+		)
+	)
+	(wire
+		(pts
 			(xy 191.77 53.34) (xy 193.04 53.34)
 		)
@@
 	(wire
 		(pts
+			(xy 229.87 33.02) (xy 231.14 33.02)
+		)
+		(stroke
+			(width 0)
+			(type default)
+		)
+	)
+	(wire
+		(pts
 			(xy 129.54 53.34) (xy 132.08 53.34)
 		)
@@
 	(wire
 		(pts
-			(xy 214.63 35.56) (xy 218.44 35.56)
-		)
-		(stroke
-			(width 0)
-			(type default)
-		)
-	)
-	(wire
-		(pts
 			(xy 162.56 88.9) (xy 166.37 88.9)
 		)
@@
 	)
 	(label "Column0"
-		(at 224.79 33.02 0)
+		(at 222.25 29.21 0)
 		(effects
 			(font
@@
 	)
 	(label "Column1"
-		(at 224.79 38.1 0)
+		(at 222.25 41.91 0)
 		(effects
 			(font
@@
 		)
 	)
-	(label "Row3"
-		(at 214.63 35.56 0)
+	(label "Row0"
+		(at 224.79 35.56 0)
 		(effects
 			(font
@@
 	(symbol
 		(lib_id "Diode:1N4148")
-		(at 222.25 35.56 0)
+		(at 226.06 33.02 0)
 		(unit 1)
 		(body_style 1)
@@
 		(dnp no)
 		(property "Reference" "D17"
-			(at 222.25 29.21 0)
+			(at 218.694 30.988 0)
 			(show_name no)
 			(do_not_autoplace no)
@@
 		)
 		(property "Value" "1N4148"
-			(at 222.25 31.75 0)
+			(at 216.916 33.782 0)
 			(show_name no)
 			(do_not_autoplace no)
@@
 		)
 		(property "Footprint" "Diode_THT:D_DO-35_SOD27_P7.62mm_Horizontal"
-			(at 222.25 35.56 0)
+			(at 226.06 33.02 0)
 			(hide yes)
 			(show_name no)
@@
 		)
 		(property "Datasheet" "https://assets.nexperia.com/documents/data-sheet/1N4148_1N4448.pdf"
-			(at 222.25 35.56 0)
+			(at 226.06 33.02 0)
 			(hide yes)
 			(show_name no)
@@
 		)
 		(property "Description" "100V 0.15A standard switching diode, DO-35"
-			(at 222.25 35.56 0)
+			(at 226.06 33.02 0)
 			(hide yes)
 			(show_name no)
@@
 		)
 		(property "Sim.Device" "D"
-			(at 222.25 35.56 0)
+			(at 226.06 33.02 0)
 			(hide yes)
 			(show_name no)
@@
 		)
 		(property "Sim.Pins" "1=K 2=A"
-			(at 222.25 35.56 0)
+			(at 226.06 33.02 0)
 			(hide yes)
 			(show_name no)
@@
 					(unit 1)
 				)
+			)
+		)
+	)
+	(symbol
+		(lib_id "Diode:1N4148")
+		(at 226.06 38.1 0)
+		(unit 1)
+		(body_style 1)
+		(exclude_from_sim no)
+		(in_bom yes)
+		(on_board yes)
+		(in_pos_files yes)
+		(dnp no)
+		(property "Reference" "D18"
+			(at 217.424 37.846 0)
+			(show_name no)
+			(do_not_autoplace no)
+			(effects
+				(font
+					(size 1.27 1.27)
+				)
+			)
+		)
+		(property "Value" "1N4148"
+			(at 216.916 39.878 0)
+			(show_name no)
+			(do_not_autoplace no)
+			(effects
+				(font
+					(size 1.27 1.27)
+				)
+			)
+		)
+		(property "Footprint" "Diode_THT:D_DO-35_SOD27_P7.62mm_Horizontal"
+			(at 226.06 38.1 0)
+			(hide yes)
+			(show_name no)
+			(do_not_autoplace no)
+			(effects
+				(font
+					(size 1.27 1.27)
+				)
+			)
+		)
+		(property "Datasheet" "https://assets.nexperia.com/documents/data-sheet/1N4148_1N4448.pdf"
+			(at 226.06 38.1 0)
+			(hide yes)
+			(show_name no)
+			(do_not_autoplace no)
+			(effects
+				(font
+					(size 1.27 1.27)
+				)
+			)
+		)
+		(property "Description" "100V 0.15A standard switching diode, DO-35"
+			(at 226.06 38.1 0)
+			(hide yes)
+			(show_name no)
+			(do_not_autoplace no)
+			(effects
+				(font
+					(size 1.27 1.27)
+				)
+			)
+		)
+		(property "Sim.Device" "D"
+			(at 226.06 38.1 0)
+			(hide yes)
+			(show_name no)
+			(do_not_autoplace no)
+			(effects
+				(font
+					(size 1.27 1.27)
+				)
+			)
+		)
+		(property "Sim.Pins" "1=K 2=A"
+			(at 226.06 38.1 0)
+			(hide yes)
+			(show_name no)
+			(do_not_autoplace no)
+			(effects
+				(font
+					(size 1.27 1.27)
+				)
+			)
+		)
+		(pin "2"
+		)
+		(pin "1"
+		)
+		(instances
+			(project "Gregory"
+				(path "/a9253a87-bc36-4b6b-9167-fe406c3e7921"
+					(reference "D18")
+					(unit 1)
+				)
