File: PCB/Gregory.kicad_pcb (KiCad board)
At the start: 2 copper layers, 109.8 x 110.8 mm, 44 parts, among them J1 Conn_01x03_Pin, SW1 SW_Push, SW10 SW_Push, SW11 SW_Push, SW12 SW_Push, SW13 SW_Push, SW14 SW_Push, SW15 SW_Push, SW16 SW_Push, SW17 RotaryEncoder, SW2 SW_Push, SW3 SW_Push, SW4 SW_Push, SW5 SW_Push, SW6 SW_Push, SW7 SW_Push, SW8 SW_Push, SW9 SW_Push, U1 MOUDLE-SEEEDUINO-XIAO, U2 ER_OLEDM0.91_1x-I2C

Commit message: Add files via upload
Parts:
- moved D13 0.34 mm to (134.7, 84.5)
- moved D12 0.28 mm to (115.4, 143.8)
Connections:
- D1 pad 1: Net-(D1-K) -> /Row0
- D1 pad 2: /Row0 -> Net-(D1-A)
- D10 pad 1: Net-(D10-K) -> /Row2
- D10 pad 2: /Row2 -> Net-(D10-A)
- D11 pad 1: Net-(D11-K) -> /Row2
- D11 pad 2: /Row2 -> Net-(D11-A)
- D12 pad 1: Net-(D12-K) -> /Row2
- D12 pad 2: /Row2 -> Net-(D12-A)
- D13 pad 1: Net-(D13-K) -> /Row3
- D13 pad 2: /Row3 -> Net-(D13-A)
- D14 pad 1: Net-(D14-K) -> /Row3
- D14 pad 2: /Row3 -> Net-(D14-A)
- D15 pad 1: Net-(D15-K) -> /Row3
- D15 pad 2: /Row3 -> Net-(D15-A)
- D16 pad 1: Net-(D16-K) -> /Row3
- D16 pad 2: /Row3 -> Net-(D16-A)
- D2 pad 1: Net-(D2-K) -> /Row0
- D2 pad 2: /Row0 -> Net-(D2-A)
- D3 pad 1: Net-(D3-K) -> /Row0
- D3 pad 2: /Row0 -> Net-(D3-A)
- D4 pad 1: Net-(D4-K) -> /Row0
- D4 pad 2: /Row0 -> Net-(D4-A)
- D5 pad 1: Net-(D5-K) -> /Row1
- D5 pad 2: /Row1 -> Net-(D5-A)
- D6 pad 1: Net-(D6-K) -> /Row1
- D6 pad 2: /Row1 -> Net-(D6-A)
- D7 pad 1: Net-(D7-K) -> /Row1
- D7 pad 2: /Row1 -> Net-(D7-A)
- D8 pad 1: Net-(D8-K) -> /Row1
- D8 pad 2: /Row1 -> Net-(D8-A)
- D9 pad 1: Net-(D9-K) -> /Row2
- D9 pad 2: /Row2 -> Net-(D9-A)
- SW1 pad 2: Net-(D1-K) -> Net-(D1-A)
- SW10 pad 2: Net-(D10-K) -> Net-(D10-A)
- SW11 pad 2: Net-(D11-K) -> Net-(D11-A)
- SW12 pad 2: Net-(D12-K) -> Net-(D12-A)
- SW13 pad 2: Net-(D13-K) -> Net-(D13-A)
- SW14 pad 2: Net-(D14-K) -> Net-(D14-A)
- SW15 pad 2: Net-(D15-K) -> Net-(D15-A)
- SW16 pad 2: Net-(D16-K) -> Net-(D16-A)
- SW2 pad 2: Net-(D2-K) -> Net-(D2-A)
- SW3 pad 2: Net-(D3-K) -> Net-(D3-A)
- SW4 pad 2: Net-(D4-K) -> Net-(D4-A)
- SW5 pad 2: Net-(D5-K) -> Net-(D5-A)
- SW6 pad 2: Net-(D6-K) -> Net-(D6-A)
- SW7 pad 2: Net-(D7-K) -> Net-(D7-A)
- SW8 pad 2: Net-(D8-K) -> Net-(D8-A)
- SW9 pad 2: Net-(D9-K) -> Net-(D9-A)
Routing:
- net Net-(D15-A): track 0.00 -> 21.3 mm
- net Net-(D16-A): track 0.00 -> 21.2 mm
- net Net-(D4-A): track 0.00 -> 21.1 mm
- net Net-(D11-A): track 0.00 -> 21.1 mm
- net Net-(D12-A): track 0.00 -> 20.8 mm
- net Net-(D6-A): track 0.00 -> 20.8 mm
- net Net-(D3-A): track 0.00 -> 20.5 mm
- net Net-(D14-A): track 0.00 -> 20.3 mm
- net Net-(D10-A): track 0.00 -> 20.3 mm
- net Net-(D13-A): track 0.00 -> 20.3 mm
- net Net-(D8-A): track 0.00 -> 20.0 mm
- net Net-(D7-A): track 0.00 -> 19.7 mm
- net Net-(D5-A): track 0.00 -> 19.4 mm
- net Net-(D2-A): track 0.00 -> 19.4 mm
- net Net-(D9-A): track 0.00 -> 19.3 mm
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