File: PCB/Gregory.kicad_sch (KiCad schematic)
At the start: 44 parts, among them J1 Conn_01x03_Pin, SW1 SW_Push, SW10 SW_Push, SW11 SW_Push, SW12 SW_Push, SW13 SW_Push, SW14 SW_Push, SW15 SW_Push, SW16 SW_Push, SW17 RotaryEncoder, SW2 SW_Push, SW3 SW_Push, SW4 SW_Push, SW5 SW_Push, SW6 SW_Push, SW7 SW_Push, SW8 SW_Push, SW9 SW_Push, U1 MOUDLE-SEEEDUINO-XIAO, U2 ER_OLEDM0.91_1x-I2C

Commit message: Add files via upload
Connections:
- net Row0: now also D1.1 (K), D2.1 (K), D3.1 (K), D4.1 (K); no longer D1.2 (A), D2.2 (A), D3.2 (A), D4.2 (A)
- net Row1: now also D5.1 (K), D6.1 (K), D7.1 (K), D8.1 (K); no longer D5.2 (A), D6.2 (A), D7.2 (A), D8.2 (A)
- net Row2: now also D10.1 (K), D11.1 (K), D12.1 (K), D9.1 (K); no longer D10.2 (A), D11.2 (A), D12.2 (A), D9.2 (A)
- net Row3: now also D13.1 (K), D14.1 (K), D15.1 (K), D16.1 (K); no longer D13.2 (A), D14.2 (A), D15.2 (A), D16.2 (A)
- net at SW5.2: now also D5.2 (A); no longer D5.1 (K)
- net at SW12.2: now also D12.2 (A); no longer D12.1 (K)
- net at SW15.2: now also D15.2 (A); no longer D15.1 (K)
- net at SW10.2: now also D10.2 (A); no longer D10.1 (K)
- net at SW9.2: now also D9.2 (A); no longer D9.1 (K)
- net at SW16.2: now also D16.2 (A); no longer D16.1 (K)
- net at SW8.2: now also D8.2 (A); no longer D8.1 (K)
- net at SW4.2: now also D4.2 (A); no longer D4.1 (K)
- net at SW1.2: now also D1.2 (A); no longer D1.1 (K)
- net at SW6.2: now also D6.2 (A); no longer D6.1 (K)
- net at SW2.2: now also D2.2 (A); no longer D2.1 (K)
- net at SW3.2: now also D3.2 (A); no longer D3.1 (K)
- net at SW7.2: now also D7.2 (A); no longer D7.1 (K)
- net at SW13.2: now also D13.2 (A); no longer D13.1 (K)
- net at SW14.2: now also D14.2 (A); no longer D14.1 (K)
- net at SW11.2: now also D11.2 (A); no longer D11.1 (K)
Other:
- moved on the sheet: D1, D10, D11, D12, D13, D14, D15, D16, D17, D18, D2, D3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
